File: hw/v1/CellShaper.kicad_pcb (KiCad board)
At the start: 4 copper layers, 100 x 100 mm, 172 parts, among them J101 Conn_01x03, J102 Conn_01x03, J103 USB_B_Micro, J104 Screw_Terminal_01x02, J105 Conn_01x03, Q201 Q_NMOS_GDS, Q202 Q_NMOS_GDS, Q203 Q_NMOS_GDS, Q301 Q_NMOS_GDS, Q302 Q_NMOS_GDS, Q303 Q_NMOS_GDS, Q401 Q_NMOS_GDS, Q402 Q_NMOS_GDS, Q403 Q_NMOS_GDS, Q501 Q_NMOS_GDS, Q502 Q_NMOS_GDS, Q503 Q_NMOS_GDS, U101 STM32F100RCTx, U101 TLV71333PDBV, U201 OPA1604, U301 OPA1604, U401 OPA1604, U501 OPA1604

Commit message: Progress with the schema and PCB....
Parts:
- removed C101, C102, C103, C104, C105, C106, C107, C108, C210, C310, C410, C510: 100n, Capacitor_SMD:C_0603_1608Metric
- removed the C408 at (151.6, 57.1)
- removed C509: 10n, Capacitor_SMD:C_0603_1608Metric
- removed the D202 at (105.0, 90.7)
- removed the D302 at (130.5, 90.7)
- removed the D402 at (153.2, 90.0)
- removed D502: D_Schottky, Diode_SMD:D_0603_1608Metric
- removed J101, J102, J105: Conn_01x03, Connector_PinHeader_2.54mm:PinHeader_1x03_P2.54mm_Horizontal
- removed J103: USB_B_Micro, Connector_USB:USB_Micro-B_Wuerth_629105150521
- removed J104: Screw_Terminal_01x02, TerminalBlock:TerminalBlock_bornier-2_P5.08mm
- removed L501: 10u, Inductor_SMD:L_Vishay_IHLP-2525
- removed Q501: Q_NMOS_GDS, Package_TO_SOT_SMD:SOT-223
- removed the R211 at (89.9, 36.8)
- removed the R213 at (105.9, 28.3)
- removed the R315 at (117.4, 67.4)
- removed the R317 at (131.2, 62.8)
- removed the R410 at (139.8, 57.7)
- removed the R415 at (143.4, 68.2)
- removed the R417 at (140.2, 70.5)
- removed R515: 150, Resistor_SMD:R_0603_1608Metric
- removed R517: 2k, Resistor_SMD:R_0603_1608Metric
- removed U101: STM32F100RCTx, Package_QFP:LQFP-48_7x7mm_P0.5mm
- removed U101: TLV71333PDBV, Package_TO_SOT_SMD:SOT-23-5
- added C308: 100n, Capacitor_SMD:C_0603_1608Metric, B.Cu at (153.3, 59.0)
- added C501: 100n, Capacitor_SMD:C_0603_1608Metric, B.Cu at (117.2, 94.8)
- added C609: 470p, Capacitor_SMD:C_0603_1608Metric, B.Cu at (172.1, 107.4)
- added C610: 470p, Capacitor_SMD:C_0603_1608Metric, B.Cu at (172.1, 110.5)
- added C611: 10u, Capacitor_SMD:C_0805_2012Metric, B.Cu at (169.9, 107.9)
- added C612: 100n, Capacitor_SMD:C_0603_1608Metric, B.Cu at (162.8, 111.0)
- added C613: 1u, Capacitor_SMD:C_0603_1608Metric, B.Cu at (164.6, 112.3)
- added C614: 100n, Capacitor_SMD:C_0603_1608Metric, B.Cu at (168.2, 108.0)
- added C701: 1u, Capacitor_SMD:C_0603_1608Metric, B.Cu at (124.8, 106.7)
- added C702: 100n, Capacitor_SMD:C_0603_1608Metric, B.Cu at (137.6, 117.8)
- added C703: 100n, Capacitor_SMD:C_0603_1608Metric, B.Cu at (143.2, 105.8)
- added C704: 100n, Capacitor_SMD:C_0603_1608Metric, B.Cu at (125.8, 107.7)
- added C705: 100n, Capacitor_SMD:C_0603_1608Metric, B.Cu at (130.6, 101.8)
- added C706: 100n, Capacitor_SMD:C_0603_1608Metric, B.Cu at (118.2, 111.0)
- added C707: 100n, Capacitor_SMD:C_0603_1608Metric, B.Cu at (126.4, 111.8)
- added C708: 10n, Capacitor_SMD:C_0603_1608Metric, B.Cu at (150.3, 109.8)
- added C712: 100n, Capacitor_SMD:C_0603_1608Metric, B.Cu at (114.8, 104.2)
- added C713: 1u, Capacitor_SMD:C_0603_1608Metric, B.Cu at (154.0, 107.1)
- added C714: 1u, Capacitor_SMD:C_0603_1608Metric, B.Cu at (148.4, 107.1)
- added D203: DFLS230Q, Diode_SMD:D_PowerDI-123, B.Cu at (97.3, 85.8)
- added D303: DFLS230Q, Diode_SMD:D_PowerDI-123, B.Cu at (147.7, 85.8)
- added D403: DFLS230Q, Diode_SMD:D_PowerDI-123, B.Cu at (173.2, 85.9)
- added D603: DFLS230Q, Diode_SMD:D_PowerDI-123, B.Cu at (122.4, 86.1)
- added D604: D, Diode_SMD:D_SOD-123, B.Cu at (161.2, 103.2)
- added D605: D, Diode_SMD:D_SOD-123, B.Cu at (158.8, 103.2)
- added D608: 3.6V, Diode_SMD:D_SOD-110, B.Cu at (150.2, 102.7)
- added H5: M3 hole, MountingHole:MountingHole_3.2mm_M3_Pad, F.Cu at (135.0, 61.0)
- added H6: M3 hole, MountingHole:MountingHole_3.2mm_M3_Pad, F.Cu at (135.0, 141.0)
- added J502: USB_C_Receptacle, Connector_USB:USB_C_Receptacle_Amphenol_12401610E4-2A, B.Cu at (180.0, 109.0)
- added J601: Screw_Terminal, TerminalBlock:TerminalBlock_bornier-2_P5.08mm, B.Cu at (181.8, 97.0)
- added J602: USB_B_Micro, Connector_USB:USB_Micro-B_GCT_USB3076-30-A, B.Cu at (182.3, 121.3)
- added J701: SWD connector, Connector_PinHeader_2.54mm:PinHeader_1x03_P2.54mm_Vertical, F.Cu at (135.0, 133.5)
- added J702: Conn_01x03, Connector_PinHeader_2.54mm:PinHeader_1x03_P2.54mm_Horizontal, B.Cu at (86.9, 129.0)
- added J703: Conn_01x03, Connector_PinHeader_2.54mm:PinHeader_1x03_P2.54mm_Horizontal, B.Cu at (183.6, 134.1)
- added L601: 100u, Inductor_SMD:L_Wuerth_HCI-7050, B.Cu at (128.8, 83.2)
- added LOGO1: Logo_Open_Hardware_Small, Symbol:OSHW-Logo_7.5x8mm_SilkScreen, B.Cu at (106.4, 111.3)
- added LOGO2: Logo_Open_Hardware_Small, Symbol:OSHW-Logo_7.5x8mm_SilkScreen, F.Cu at (135.1, 109.3)
- added NT1: Net-Tie_2, NetTie:NetTie-2_SMD_Pad2.0mm, F.Cu at (165.4, 99.5)
- added Q601: ZVN4206G, Package_TO_SOT_SMD:SOT-223-3_TabPin2, B.Cu at (128.1, 91.1)
- added R218: 100k, Resistor_SMD:R_0603_1608Metric, B.Cu at (93.2, 67.0)
- added R219: 10k, Resistor_SMD:R_0603_1608Metric, B.Cu at (105.5, 57.9)
- added R220: 0, Resistor_SMD:R_0603_1608Metric, B.Cu at (96.5, 93.2)
- added R311: 1k 0.5%, Resistor_SMD:R_0603_1608Metric, B.Cu at (142.8, 50.8)
- added R318: 100k, Resistor_SMD:R_0603_1608Metric, B.Cu at (144.5, 65.9)
- added R319: 10k, Resistor_SMD:R_0603_1608Metric, B.Cu at (153.3, 57.5)
- added R320: 0, Resistor_SMD:R_0603_1608Metric, B.Cu at (146.6, 93.1)
- added R418: 100k, Resistor_SMD:R_0603_1608Metric, B.Cu at (167.7, 66.8)
- added R419: 10k, Resistor_SMD:R_0603_1608Metric, B.Cu at (176.3, 57.9)
- added R420: 0, Resistor_SMD:R_0603_1608Metric, B.Cu at (172.6, 92.8)
- added R501: 0, Resistor_SMD:R_0603_1608Metric, B.Cu at (121.2, 93.3)
- added R618: 100k, Resistor_SMD:R_0603_1608Metric, B.Cu at (118.9, 66.7)
- added R619: 10k, Resistor_SMD:R_0603_1608Metric, B.Cu at (128.0, 58.1)
- added R620: 4k7, Resistor_SMD:R_0603_1608Metric, B.Cu at (151.2, 112.9)
- added R621: 4k7, Resistor_SMD:R_0603_1608Metric, B.Cu at (152.7, 112.9)
- added R622: 4k7, Resistor_SMD:R_0603_1608Metric, B.Cu at (154.2, 112.9)
- added R623: 100k, Resistor_SMD:R_0603_1608Metric, B.Cu at (153.4, 102.7)
- added R624: 27k, Resistor_SMD:R_0603_1608Metric, B.Cu at (151.9, 102.7)
- added R625: 0, Resistor_SMD:R_0603_1608Metric, B.Cu at (176.6, 115.7)
- added R626: 10k, Resistor_SMD:R_0603_1608Metric, B.Cu at (174.9, 97.2)
- added R701: 10k, Resistor_SMD:R_0603_1608Metric, B.Cu at (127.9, 113.6)
- added R702: 10k, Resistor_SMD:R_0603_1608Metric, B.Cu at (134.5, 96.0)
- added R703: 10k, Resistor_SMD:R_0603_1608Metric, B.Cu at (134.5, 97.5)
- added TH201: Thermistor_NTC, CellShaper:ContactThermistor, F.Cu at (97.4, 115.0)
- added TH301: Thermistor_NTC, CellShaper:ContactThermistor, F.Cu at (147.5, 115.0)
- added TH401: Thermistor_NTC, CellShaper:ContactThermistor, F.Cu at (172.5, 115.0)
- added TH601: Thermistor_NTC, CellShaper:ContactThermistor, F.Cu at (122.4, 115.0)
- added TH701: 10k_NTC, Resistor_SMD:R_0603_1608Metric, B.Cu at (134.5, 94.5)
- added TH702: 10k_NTC, Connector_PinHeader_1.27mm:PinHeader_1x02_P1.27mm_Vertical, F.Cu at (134.3, 54.5)
- added TP601: TestPoint, TestPoint:TestPoint_Pad_D1.5mm, B.Cu at (169.2, 110.9)
- added U202: LMV344IPWR, Package_SO:TSSOP-14_4.4x5mm_P0.65mm, B.Cu at (99.0, 61.9)
- added U302: LMV344IPWR, Package_SO:TSSOP-14_4.4x5mm_P0.65mm, B.Cu at (147.5, 61.6)
- added U402: LMV344IPWR, Package_SO:TSSOP-14_4.4x5mm_P0.65mm, B.Cu at (170.8, 61.4)
- added U502: LMV344IPWR, Package_SO:TSSOP-14_4.4x5mm_P0.65mm, B.Cu at (122.4, 62.1)
- added U602: FUSB302BMPX, Package_DFN_QFN:WQFN-14-1EP_2.5x2.5mm_P0.5mm_EP1.45x1.45mm, B.Cu at (165.6, 108.9)
- added U701: STM32F303RBTx, Package_QFP:LQFP-64_10x10mm_P0.5mm, B.Cu at (135.0, 109.0)
- added U702: DAC084S085, Package_SO:VSSOP-10_3x3mm_P0.5mm, B.Cu at (117.3, 106.7)
- added U703: LP2985-3.3, Package_TO_SOT_SMD:SOT-23-5, B.Cu at (151.3, 107.2)
- added Y701: 8MHz crystal, Crystal:Crystal_SMD_Abracon_ABM8G-4Pin_3.2x2.5mm, B.Cu at (127.8, 104.1)
- C201, C202: value 10u -> 10u 16V
- C204: renamed from C203; value 10u -> 22u
- C205: renamed from C204; value 1u -> 10u
- C209, C309, C409: value 10n -> 100n
- C301: renamed from C401; value 10u -> 10u 16V
- C302: renamed from C402; value 10u -> 10u 16V
- C304: renamed from C403; value 10u -> 22u
- C305: renamed from C404; value 1u -> 10u
- C401: renamed from C501; value 10u -> 10u 16V
- C402: renamed from C502; value 10u -> 10u 16V
- C404: renamed from C503; value 10u -> 22u
- C405: renamed from C504; value 1u -> 10u
- C601: renamed from C301; value 10u -> 10u 16V
- C602: renamed from C302; value 10u -> 10u 16V
- C604: renamed from C303; value 10u -> 22u
- C605: renamed from C304; value 1u -> 10u
- L201, L301, L401: value 10u -> 100u; footprint Inductor_SMD:L_Vishay_IHLP-2525 -> Inductor_SMD:L_Wuerth_HCI-7050
- Q201, Q301, Q401: value Q_NMOS_GDS -> ZVN4206G; footprint Package_TO_SOT_SMD:SOT-223 -> Package_TO_SOT_SMD:SOT-223-3_TabPin2
- Q202, Q203: value Q_NMOS_GDS -> IRFZ24NPbF
- Q302: renamed from Q402; value Q_NMOS_GDS -> IRFZ24NPbF
- Q303: renamed from Q403; value Q_NMOS_GDS -> IRFZ24NPbF
- Q402: renamed from Q502; value Q_NMOS_GDS -> IRFZ24NPbF
- Q403: renamed from Q503; value Q_NMOS_GDS -> IRFZ24NPbF
- Q602: renamed from Q302; value Q_NMOS_GDS -> IRFZ24NPbF
- Q603: renamed from Q303; value Q_NMOS_GDS -> IRFZ24NPbF
- R203: renamed from R201; value R -> 10k
- R204: renamed from R202; value 1k -> 22k 0.5%
- R205: renamed from R203; value 1k -> 1k 0.5%
- R206: renamed from R204; value 0R1 -> 0R1 1%
- R207: renamed from R205; value 1k -> 1k 0.5%
- R208: renamed from R219; value 1k -> 22k 0.5%
- R209: renamed from R218; value R -> 10k
- R210: renamed from R206; value 0R1 -> 0R1 1%
- R211: renamed from R208; value 1k -> 1k 0.5%
- R212: renamed from R209; value 1k -> 1k 0.5%
- R213: renamed from R207; value 1k -> 100
- R214: renamed from R210; value 1k -> 200k
- R215: value 2k -> 1k
- R216: renamed from R212; value 1k -> 22k 0.5%
- R217: renamed from R214; value 18k -> 1k
- R303: renamed from R403; value R -> 10k
- R304: renamed from R404; value 1k -> 22k 0.5%
- R305: renamed from R405; value 1k -> 1k 0.5%
- R306: renamed from R406; value 0R1 -> 0R1 1%
- R307: renamed from R407; value 1k -> 1k 0.5%
- R308: renamed from R419; value 1k -> 22k 0.5%
- R309: renamed from R418; value R -> 10k
- R310: renamed from R408; value 0R1 -> 0R1 1%
- R312: renamed from R411; value 1k -> 1k 0.5%
- R313: renamed from R409; value 1k -> 100
- R314: renamed from R412; value 1k -> 200k
- R316: renamed from R414; value 1k -> 22k 0.5%
- R317: renamed from R416; value 18k -> 1k
- R403: renamed from R503; value R -> 10k
- R404: renamed from R504; value 1k -> 22k 0.5%
- R405: renamed from R505; value 1k -> 1k 0.5%
- R406: renamed from R506; value 0R1 -> 0R1 1%
- R407: renamed from R507; value 1k -> 1k 0.5%
- R408: renamed from R519; value 1k -> 22k 0.5%
- R409: renamed from R518; value R -> 10k
- R410: renamed from R508; value 0R1 -> 0R1 1%
- R411: renamed from R510; value 1k -> 1k 0.5%
- R412: renamed from R511; value 1k -> 1k 0.5%
- R413: renamed from R509; value 1k -> 100
- R414: renamed from R512; value 1k -> 200k
- R416: renamed from R514; value 1k -> 22k 0.5%
- R417: renamed from R516; value 18k -> 1k
- R603: renamed from R303; value R -> 10k
- R604: renamed from R304; value 1k -> 22k 0.5%
- R605: renamed from R305; value 1k -> 1k 0.5%
- R606: renamed from R306; value 0R1 -> 0R1 1%
- R607: renamed from R307; value 1k -> 1k 0.5%
- R608: renamed from R319; value 1k -> 22k 0.5%
- R609: renamed from R318; value R -> 10k
- R610: renamed from R308; value 0R1 -> 0R1 1%
- R611: renamed from R310; value 1k -> 1k 0.5%
- R612: renamed from R311; value 1k -> 1k 0.5%
- R613: renamed from R309; value 1k -> 100
- R614: renamed from R312; value 1k -> 200k
- R616: renamed from R314; value 1k -> 22k 0.5%
- R617: renamed from R316; value 18k -> 1k
- U201, U301, U401, U501: value OPA1604 -> MCP1416; footprint Package_SO:SOIC-16_3.9x9.9mm_P1.27mm -> Package_TO_SOT_SMD:SOT-23-5
- moved R203 64.7 mm to (92.8, 89.1), turned to 0 degrees
- moved R403 63.3 mm to (167.9, 88.8), turned to 0 degrees
- moved U501 59.7 mm to (117.6, 92.2), turned to 0 degrees
- moved C209 56.8 mm to (92.4, 94.5), turned to 0 degrees
- moved R217 47.5 mm to (90.0, 74.3), turned to 270 degrees
- moved R404 43.8 mm to (174.9, 66.2), turned to 270 degrees
- moved R207 43.3 mm to (102.2, 68.8), turned to 270 degrees
- moved C309 42.4 mm to (142.6, 94.7), turned to 0 degrees
- moved R407 42.2 mm to (176.6, 68.0), turned to 270 degrees
- moved C406 41.5 mm to (177.3, 65.7), turned to 0 degrees
- moved R204 40.6 mm to (100.6, 66.3), turned to 270 degrees
- moved C409 38.9 mm to (165.3, 92.2), turned to 270 degrees
- moved R417 36.8 mm to (165.2, 77.3), turned to 270 degrees
- moved C206 36.5 mm to (103.0, 66.5), turned to 0 degrees
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- renumbered BT401 to BT301, BT501 to BT401, BT301 to BT601, C206 to C203, C205 to C206, C406 to C303, C405 to C306, C407 to C307, C506 to C403, C505 to C406, C507 to C407, C508 to C408, C306 to C603, C305 to C606, C307 to C607, C308 to C608, D203 to D202, D401 to D301, D403 to D302, D501 to D401, D503 to D402, D301 to D601, D303 to D602, HS101 to HS1, R216 to R201, R217 to R202, R401 to R301, R402 to R302, R413 to R315, R501 to R401, R502 to R402, R513 to R415, R301 to R601, R302 to R602, R313 to R615
Connections:
- BT201 pad 1: /Cell_A/CELL -> /Cell_A/CELL_POSITIVE
- BT201 pad 2: GND -> GNDPWR
- BT301 pad 1: /Cell_C/CELL -> /Cell_C/CELL_POSITIVE
- BT301 pad 2: GND -> GNDPWR
- BT401 pad 1: /Cell_D/CELL -> /Cell_D/CELL_POSITIVE
- BT401 pad 2: GND -> GNDPWR
- BT601 pad 1: /Cell_B/CELL -> /Cell_B/CELL_POSITIVE
- BT601 pad 2: GND -> GNDPWR
- C206 pad 1: Net-(C205-Pad1) -> Net-(C206-Pad1)
- C206 pad 2: Net-(C205-Pad2) -> Net-(C206-Pad2)
- C209 pad 1: Net-(C209-Pad1) -> /CHARGE_POWER
- C304 pad 1: Net-(C403-Pad1) -> Net-(C304-Pad1)
- C305 pad 1: Net-(C403-Pad1) -> Net-(C304-Pad1)
- C306 pad 1: Net-(C405-Pad1) -> Net-(C306-Pad1)
- C306 pad 2: Net-(C405-Pad2) -> Net-(C306-Pad2)
- C307 pad 1: Net-(C407-Pad1) -> Net-(C307-Pad1)
- C307 pad 2: Net-(C407-Pad2) -> Net-(C307-Pad2)
- C309 pad 1: Net-(C309-Pad1) -> /CHARGE_POWER
- C404 pad 1: Net-(C503-Pad1) -> Net-(C404-Pad1)
- C405 pad 1: Net-(C503-Pad1) -> Net-(C404-Pad1)
- C406 pad 1: Net-(C505-Pad1) -> Net-(C406-Pad1)
- C406 pad 2: Net-(C505-Pad2) -> Net-(C406-Pad2)
- C407 pad 1: Net-(C507-Pad1) -> Net-(C407-Pad1)
- C407 pad 2: Net-(C507-Pad2) -> Net-(C407-Pad2)
- C408 pad 1: Net-(C508-Pad1) -> Net-(C408-Pad1)
- C409 pad 1: Net-(C409-Pad1) -> /CHARGE_POWER
- C604 pad 1: Net-(C303-Pad1) -> Net-(C604-Pad1)
- C605 pad 1: Net-(C303-Pad1) -> Net-(C604-Pad1)
- C606 pad 1: Net-(C305-Pad1) -> Net-(C606-Pad1)
- C606 pad 2: Net-(C305-Pad2) -> Net-(C606-Pad2)
- C607 pad 1: Net-(C307-Pad1) -> Net-(C607-Pad1)
- C607 pad 2: Net-(C307-Pad2) -> Net-(C607-Pad2)
- C608 pad 1: Net-(C308-Pad1) -> Net-(C608-Pad1)
- L301 pad 2: Net-(C303-Pad1) -> Net-(C304-Pad1)
- L401 pad 2: Net-(C403-Pad1) -> Net-(C404-Pad1)
- Q201 pad 1: /CELL_A_CHARGE -> /Cell_A/GATE
- Q202 pad 2: /Cell_A/CELL -> /Cell_A/CELL_POSITIVE
- Q203 pad 2: /Cell_A/CELL -> /Cell_A/CELL_POSITIVE
- Q301 pad 1: /CELL_B_CHARGE -> /Cell_C/GATE
- Q302 pad 2: /Cell_C/CELL -> /Cell_C/CELL_POSITIVE
- Q303 pad 2: /Cell_C/CELL -> /Cell_C/CELL_POSITIVE
- Q401 pad 1: /CELL_C_CHARGE -> /Cell_D/GATE
- Q402 pad 2: /Cell_D/CELL -> /Cell_D/CELL_POSITIVE
- Q403 pad 2: /Cell_D/CELL -> /Cell_D/CELL_POSITIVE
- Q602 pad 2: /Cell_B/CELL -> /Cell_B/CELL_POSITIVE
- Q603 pad 2: /Cell_B/CELL -> /Cell_B/CELL_POSITIVE
- R201 pad 1: /CELL_A_CHARGE_LED -> /MCU/CELL_A_CHARGE_LED
- R202 pad 1: /CELL_A_DISCHARGE_LED -> /MCU/CELL_A_DISCHARGE_LED
- R203 pad 1: /CELL_A_CHARGE -> /MCU/CELL_A_CHARGE
- R204 pad 1: /CELL_A_CHARGE_CURRENT -> /MCU/CELL_A_CHARGE_CURRENT
- R204 pad 2: Net-(C205-Pad2) -> Net-(C206-Pad1)
- R205 pad 1: Net-(C205-Pad2) -> Net-(C206-Pad2)
- R206 pad 2: /Cell_A/CELL -> /Cell_A/CELL_POSITIVE
- R207 pad 1: Net-(C205-Pad1) -> Net-(C206-Pad1)
- R207 pad 2: /Cell_A/CELL -> /Cell_A/CELL_POSITIVE
- R208 pad 2: Net-(C205-Pad1) -> Net-(C206-Pad2)
- R209 pad 1: /CELL_A_TEMPERATURE -> +3V3
- R209 pad 2: GND -> /MCU/CELL_A_TEMPERATURE
- R210 pad 2: GND -> GNDPWR
- R212 pad 1: GND -> GNDPWR
- R214 pad 1: /Cell_A/CELL -> Net-(R214-Pad1)
- R214 pad 2: Net-(R210-Pad2) -> GNDPWR
- R215 pad 1: /CELL_A_DISCHARGE -> Net-(C208-Pad2)
- R215 pad 2: GND -> /MCU/CELL_A_DISCHARGE_CURRENT
- R216 pad 2: /CELL_A_DISCHARGE_CURRENT -> /MCU/CELL_A_DISCHARGE_CURRENT
- R217 pad 1: Net-(C209-Pad1) -> Net-(R217-Pad1)
- R217 pad 2: /CELL_A_DISCHARGE -> /MCU/CELL_A_DISCHARGE
- R301 pad 1: /CELL_C_CHARGE_LED -> /MCU/CELL_C_CHARGE_LED
- R302 pad 1: /CELL_C_DISCHARGE_LED -> /MCU/CELL_C_DISCHARGE_LED
- R303 pad 1: /CELL_C_CHARGE -> /MCU/CELL_C_CHARGE
- R304 pad 1: /CELL_C_CHARGE_CURRENT -> /MCU/CELL_C_CHARGE_CURRENT
- R304 pad 2: Net-(C405-Pad2) -> Net-(C306-Pad1)
- R305 pad 1: Net-(C405-Pad2) -> Net-(C306-Pad2)
- R305 pad 2: Net-(C403-Pad1) -> Net-(C304-Pad1)
- R306 pad 1: Net-(C403-Pad1) -> Net-(C304-Pad1)
- R306 pad 2: /Cell_C/CELL -> /Cell_C/CELL_POSITIVE
- R307 pad 1: Net-(C405-Pad1) -> Net-(C306-Pad1)
- R307 pad 2: /Cell_C/CELL -> /Cell_C/CELL_POSITIVE
- R308 pad 2: Net-(C405-Pad1) -> Net-(C306-Pad2)
- R309 pad 1: /CELL_C_TEMPERATURE -> +3V3
- R309 pad 2: GND -> /MCU/CELL_C_TEMPERATURE
- R310 pad 2: GND -> GNDPWR
- R312 pad 1: GND -> GNDPWR
- R312 pad 2: Net-(C407-Pad1) -> Net-(C307-Pad1)
- R313 pad 2: Net-(C408-Pad1) -> Net-(C308-Pad1)
- R314 pad 1: /Cell_C/CELL -> Net-(R314-Pad1)
- R314 pad 2: Net-(R412-Pad2) -> GNDPWR
- R315 pad 2: /CELL_C_DISHARGE_CURRENT -> /MCU/CELL_C_DISCHARGE_CURRENT
- R316 pad 1: Net-(C407-Pad1) -> Net-(C307-Pad1)
- R316 pad 2: /CELL_C_DISHARGE_CURRENT -> /MCU/CELL_C_DISCHARGE_CURRENT
- R317 pad 1: Net-(C409-Pad1) -> Net-(R317-Pad1)
- R317 pad 2: /CELL_C_DISCHARGE -> /MCU/CELL_C_DISCHARGE
- R401 pad 1: /CELL_D_CHARGE_LED -> /MCU/CELL_D_CHARGE_LED
- R402 pad 1: /CELL_D_DISCHARGE_LED -> /MCU/CELL_D_DISCHARGE_LED
- R403 pad 1: /CELL_D_CHARGE -> /MCU/CELL_D_CHARGE
- R404 pad 1: /CELL_D_CHARGE_CURRENT -> /MCU/CELL_D_DISCHARGE_CURRENT
- R404 pad 2: Net-(C505-Pad2) -> Net-(C406-Pad1)
- R405 pad 1: Net-(C505-Pad2) -> Net-(C406-Pad2)
- R405 pad 2: Net-(C503-Pad1) -> Net-(C404-Pad1)
- R406 pad 1: Net-(C503-Pad1) -> Net-(C404-Pad1)
- R406 pad 2: /Cell_D/CELL -> /Cell_D/CELL_POSITIVE
- R407 pad 1: Net-(C505-Pad1) -> Net-(C406-Pad1)
- R407 pad 2: /Cell_D/CELL -> /Cell_D/CELL_POSITIVE
- R408 pad 2: Net-(C505-Pad1) -> Net-(C406-Pad2)
- R409 pad 1: /CELL_D_TEMPERATURE -> +3V3
- R409 pad 2: GND -> /MCU/CELL_D_TEMPERATURE
- R410 pad 2: GND -> GNDPWR
- R411 pad 2: Net-(C507-Pad2) -> Net-(C407-Pad2)
- R412 pad 1: GND -> GNDPWR
- R412 pad 2: Net-(C507-Pad1) -> Net-(C407-Pad1)
- R413 pad 2: Net-(C508-Pad1) -> Net-(C408-Pad1)
- R414 pad 1: /Cell_D/CELL -> Net-(R414-Pad1)
- R414 pad 2: Net-(R512-Pad2) -> GNDPWR
- R415 pad 2: /CELL_D_DISCHARGE_CURRENT -> /MCU/CELL_D_CHARGE_CURRENT
- R416 pad 1: Net-(C507-Pad1) -> Net-(C407-Pad1)
- R416 pad 2: /CELL_D_DISCHARGE_CURRENT -> /MCU/CELL_D_CHARGE_CURRENT
- R417 pad 1: Net-(C509-Pad1) -> Net-(R417-Pad1)
- R417 pad 2: /CELL_D_DISCHARGE -> /MCU/CELL_D_DISCHARGE
- R601 pad 1: /CELL_B_CHARGE_LED -> /MCU/CELL_B_CHARGE_LED
- R602 pad 1: /CELL_B_DISCHARGE_LED -> /MCU/CELL_B_DISCHARGE_LED
- R603 pad 1: /CELL_B_CHARGE -> /MCU/CELL_B_CHARGE
- R604 pad 1: /CELL_B_CHARGE_CURRENT -> /MCU/CELL_B_CHARGE_CURRENT
- R604 pad 2: Net-(C305-Pad2) -> Net-(C606-Pad1)
- R605 pad 1: Net-(C305-Pad2) -> Net-(C606-Pad2)
- R605 pad 2: Net-(C303-Pad1) -> Net-(C604-Pad1)
- R606 pad 1: Net-(C303-Pad1) -> Net-(C604-Pad1)
- R606 pad 2: /Cell_B/CELL -> /Cell_B/CELL_POSITIVE
- R607 pad 1: Net-(C305-Pad1) -> Net-(C606-Pad1)
- R607 pad 2: /Cell_B/CELL -> /Cell_B/CELL_POSITIVE
- R608 pad 2: Net-(C305-Pad1) -> Net-(C606-Pad2)
- R609 pad 1: /CELL_B_TEMPERATURE -> +3V3
- R609 pad 2: GND -> /MCU/CELL_B_TEMPERATURE
- R610 pad 2: GND -> GNDPWR
- R611 pad 2: Net-(C307-Pad2) -> Net-(C607-Pad2)
- R612 pad 1: GND -> GNDPWR
- R612 pad 2: Net-(C307-Pad1) -> Net-(C607-Pad1)
- R613 pad 2: Net-(C308-Pad1) -> Net-(C608-Pad1)
- R614 pad 1: /Cell_B/CELL -> Net-(R614-Pad1)
- R614 pad 2: Net-(R312-Pad2) -> GNDPWR
- R615 pad 2: /CELL_B_DISCHARGE_CURRENT -> /MCU/CELL_B_DISCHARGE_CURRENT
- R616 pad 1: Net-(C307-Pad1) -> Net-(C607-Pad1)
- R616 pad 2: /CELL_B_DISCHARGE_CURRENT -> /MCU/CELL_B_DISCHARGE_CURRENT
- R617 pad 1: Net-(C309-Pad1) -> Net-(R617-Pad1)
- R617 pad 2: /CELL_B_DISCHARGE -> /MCU/CELL_B_DISCHARGE
- U201 pad 1: /CELL_A_DISCHARGE_CURRENT -> Net-(U201-Pad1)
- U201 pad 2: Net-(C207-Pad1) -> /CHARGE_POWER
- U201 pad 3: Net-(C207-Pad2) -> /MCU/CELL_A_CHARGE
- U201 pad 4: +5V -> GND
- U201 pad 5: Net-(C209-Pad1) -> Net-(R220-Pad2)
- U301 pad 1: /CELL_B_DISCHARGE_CURRENT -> Net-(U301-Pad1)
- U301 pad 2: Net-(C307-Pad1) -> /CHARGE_POWER
- U301 pad 3: Net-(C307-Pad2) -> /MCU/CELL_C_CHARGE
- U301 pad 4: +5V -> GND
- U301 pad 5: Net-(C309-Pad1) -> Net-(R320-Pad2)
- U401 pad 1: /CELL_C_DISHARGE_CURRENT -> Net-(U401-Pad1)
- U401 pad 2: Net-(C407-Pad1) -> /CHARGE_POWER
- U401 pad 3: Net-(C407-Pad2) -> /MCU/CELL_D_CHARGE
- U401 pad 4: +5V -> GND
- U401 pad 5: Net-(C409-Pad1) -> Net-(R420-Pad2)
- U501 pad 1: /CELL_D_DISCHARGE_CURRENT -> Net-(U501-Pad1)
- U501 pad 2: Net-(C507-Pad1) -> /CHARGE_POWER
- U501 pad 3: Net-(C507-Pad2) -> /MCU/CELL_B_CHARGE
- U501 pad 4: +5V -> GND
- U501 pad 5: Net-(C509-Pad1) -> Net-(R501-Pad2)
Routing:
- net GND: track 7.39 -> 240.6 mm, vias 4 -> 40
- net /MCU/TXD: track 0.00 -> 127.3 mm, vias 0 -> 4
- net /MCU/RXD: track 0.00 -> 126.7 mm, vias 0 -> 2
- net GNDPWR: track 0.00 -> 114.3 mm, vias 0 -> 53
- net /CHARGE_POWER: track 83.0 -> 6.22 mm
- net /MCU/CELL_A_VOLTAGE: track 0.00 -> 74.6 mm, vias 0 -> 2
- net /Power/DN: track 0.00 -> 68.3 mm, vias 0 -> 7
- net /MCU/CELL_D_DISCHARGE: track 0.00 -> 68.0 mm, vias 0 -> 2
- net /MCU/CELL_A_CHARGE_CURRENT: track 0.00 -> 63.3 mm, vias 0 -> 2
- net /MCU/CELL_A_DISCHARGE_CURRENT: track 0.00 -> 63.2 mm, vias 0 -> 2
- net /MCU/CELL_C_DISCHARGE: track 0.00 -> 62.2 mm, vias 0 -> 2
- net /Power/DP: track 0.00 -> 60.1 mm, vias 0 -> 5
- net /MCU/CELL_D_DISCHARGE_LED: track 0.00 -> 54.8 mm
- net /MCU/CELL_D_CHARGE_LED: track 0.00 -> 53.7 mm
- net /MCU/CELL_D_CHARGE_CURRENT: track 0.00 -> 53.4 mm
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- added copper zone on In1.Cu, net +3V3
- added copper zone on In1.Cu, net /CHARGE_POWER
- added copper zone on In1.Cu, net /Power/USB_VBUS
- added copper zone on In1.Cu, net GNDPWR
- added copper zone on In2.Cu, net GNDPWR
Other:
- board text added: "- +"
- board text added: "A"
- board text added: "B"
- board text added: "C"
- board text added: "CellShaper v1"
- board text added: "D"
- board text added: "DC 5-12V"
- board text added: "SWDIO SWCLK GND"
- board text added: "petrinm"

Commit message: Progress...
Parts:
- added C709: 1u, Capacitor_SMD:C_0603_1608Metric, B.Cu at (154.0, 106.5)
- added C710: 10n, Capacitor_SMD:C_0603_1608Metric, B.Cu at (149.6, 109.5)
- added C711: 1u, Capacitor_SMD:C_0603_1608Metric, B.Cu at (148.3, 107.0)
- added C715: Xp, Capacitor_SMD:C_0603_1608Metric, B.Cu at (128.6, 102.2)
- added C716: Xp, Capacitor_SMD:C_0603_1608Metric, B.Cu at (124.9, 102.7)
- added R221: 300k 0.5%, Resistor_SMD:R_0603_1608Metric, B.Cu at (94.4, 67.0)
- added R222: 300k 0.5%, Resistor_SMD:R_0603_1608Metric, B.Cu at (93.6, 63.1)
- added R223: 100k 0.5%, Resistor_SMD:R_0603_1608Metric, B.Cu at (99.8, 58.2)
- added R321: 300k 0.5%, Resistor_SMD:R_0603_1608Metric, B.Cu at (145.2, 66.3)
- added R322: 300k 0.5%, Resistor_SMD:R_0603_1608Metric, B.Cu at (141.3, 62.5)
- added R323: 100k 0.5%, Resistor_SMD:R_0603_1608Metric, B.Cu at (148.0, 57.9)
- added R421: 300k 0.5%, Resistor_SMD:R_0603_1608Metric, B.Cu at (169.0, 65.9)
- added R422: 300k 0.5%, Resistor_SMD:R_0603_1608Metric, B.Cu at (164.9, 62.4)
- added R423: 100k 0.5%, Resistor_SMD:R_0603_1608Metric, B.Cu at (172.9, 57.7)
- added R502: 300k 0.5%, Resistor_SMD:R_0603_1608Metric, B.Cu at (119.8, 66.4)
- added R503: 300k 0.5%, Resistor_SMD:R_0603_1608Metric, B.Cu at (115.5, 63.6)
- added R504: 100k 0.5%, Resistor_SMD:R_0603_1608Metric, B.Cu at (122.4, 58.1)
- added U704: LP2985-5.0, Package_TO_SOT_SMD:SOT-23-5, B.Cu at (151.2, 106.8)
- LOGO1: footprint Symbol:OSHW-Logo_7.5x8mm_SilkScreen -> Symbol:OSHW-Logo_7.5x8mm_Copper
- NT1: moved to B.Cu
- R206, R210, R306, R310, R406, R410, R606, R610: footprint Resistor_SMD:R_1210_3225Metric -> Resistor_SMD:R_1206_3216Metric
- R214, R314, R414, R614: value 200k -> 100k 0.5%
- R218, R318, R418, R618: value 100k -> 100k 0.5%
- moved J701 51.0 mm to (87.0, 116.3)
- moved R617 19.0 mm to (128.9, 62.7), turned to 0 degrees
- moved R217 18.7 mm to (105.0, 63.0), turned to 0 degrees
- moved R417 18.4 mm to (177.1, 63.2)
- moved C704 14.2 mm to (138.2, 100.6), turned to 135 degrees
- moved R212 9.05 mm to (96.0, 57.5), turned to 270 degrees
- moved D604 8.94 mm to (157.1, 111.1), turned to 0 degrees
- moved R211 8.50 mm to (97.5, 57.5), turned to 270 degrees
- moved R612 8.17 mm to (118.3, 57.5), turned to 270 degrees
- moved R312 8.00 mm to (144.0, 57.2), turned to 270 degrees
- moved R412 7.82 mm to (168.9, 57.0), turned to 270 degrees
- moved R611 7.11 mm to (119.8, 57.5), turned to 270 degrees
- moved R311 6.96 mm to (145.5, 57.2), turned to 270 degrees
- moved R411 6.85 mm to (170.4, 57.0), turned to 270 degrees
- moved TH701 6.68 mm to (128.2, 96.8), turned to 270 degrees
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Connections:
- net Net-(U701-Pad5) renamed /MCU/X1
- net Net-(U701-Pad6) renamed /MCU/X2
- C706 pad 2: Net-(C706-Pad2) -> +3V3
- HS1 pad 1: GND -> GNDPWR
- R214 pad 1: Net-(R214-Pad1) -> GND
- R214 pad 2: GNDPWR -> Net-(R214-Pad2)
- R218 pad 1: /Cell_A/CELL_POSITIVE -> /MCU/CELL_A_VOLTAGE
- R218 pad 2: Net-(R214-Pad1) -> Net-(R218-Pad2)
- R314 pad 1: Net-(R314-Pad1) -> GND
- R314 pad 2: GNDPWR -> Net-(R314-Pad2)
- R318 pad 1: /Cell_C/CELL_POSITIVE -> /MCU/CELL_C_VOLTAGE
- R318 pad 2: Net-(R314-Pad1) -> Net-(R318-Pad2)
- R414 pad 1: Net-(R414-Pad1) -> GND
- R414 pad 2: GNDPWR -> Net-(R414-Pad2)
- R418 pad 1: /Cell_D/CELL_POSITIVE -> /MCU/CELL_D_VOLTAGE
- R418 pad 2: Net-(R414-Pad1) -> Net-(R418-Pad2)
- R614 pad 1: Net-(R614-Pad1) -> GND
- R614 pad 2: GNDPWR -> Net-(R502-Pad2)
- R618 pad 1: /Cell_B/CELL_POSITIVE -> /MCU/CELL_B_VOLTAGE
- R618 pad 2: Net-(R614-Pad1) -> Net-(R503-Pad2)
- U202 pad 2: /MCU/CELL_A_VOLTAGE -> Net-(R218-Pad2)
- U202 pad 3: Net-(R214-Pad1) -> Net-(R214-Pad2)
- U302 pad 2: /MCU/CELL_C_VOLTAGE -> Net-(R318-Pad2)
- U302 pad 3: Net-(R314-Pad1) -> Net-(R314-Pad2)
- U402 pad 2: /MCU/CELL_D_VOLTAGE -> Net-(R418-Pad2)
- U402 pad 3: Net-(R414-Pad1) -> Net-(R414-Pad2)
- U502 pad 2: /MCU/CELL_B_VOLTAGE -> Net-(R503-Pad2)
- U502 pad 3: Net-(R614-Pad1) -> Net-(R502-Pad2)
- U701 pad 1: +3V3 -> Net-(U701-Pad1)
- U701 pad 15: /MCU/CELL_B_CHARGE_CURRENT -> /MCU/PCB_TEMPERATURE
- U701 pad 16: /MCU/CELL_B_DISCHARGE_CURRENT -> /MCU/HEATSINK_TEMPERATURE
- U701 pad 17: /MCU/HEATSINK_TEMPERATURE -> /MCU/CELL_B_DISCHARGE_CURRENT
- U701 pad 18: /MCU/PCB_TEMPERATURE -> /MCU/CELL_B_CHARGE_CURRENT
- U701 pad 24: /MCU/CELL_D_VOLTAGE -> /MCU/CELL_D_CHARGE_CURRENT
- U701 pad 25: /MCU/CELL_D_CHARGE_CURRENT -> /MCU/CELL_D_VOLTAGE
- U702 pad 7: Net-(C706-Pad2) -> +3V3
Routing:
- net GNDPWR: track 114.3 -> 348.9 mm, vias 53 -> 93
- net +5V: track 2.64 -> 137.1 mm, vias 1 -> 5
- net GND: track 240.6 -> 323.3 mm, vias 40 -> 96
- net /CHARGE_POWER: track 6.22 -> 86.2 mm, vias 0 -> 17
- net /MCU/SBWDIO: track 16.1 -> 62.1 mm, vias 0 -> 2
- net /MCU/CELL_C_DISCHARGE_CURRENT: track 22.8 -> 68.2 mm
- net /MCU/CELL_C_CHARGE_CURRENT: track 25.7 -> 65.7 mm
- net /MCU/CELL_B_DISCHARGE_CURRENT: track 34.9 -> 69.6 mm, vias 0 -> 2
- net /Cell_A/CELL_POSITIVE: track 24.7 -> 57.3 mm
- net /MCU/SBWCLK: track 19.8 -> 52.2 mm
- net /MCU/CELL_A_DISCHARGE_CURRENT: track 63.2 -> 92.9 mm, vias 2 -> 5
- net /MCU/CELL_B_DISCHARGE: track 32.1 -> 58.1 mm
- net /MCU/CELL_D_CHARGE_CURRENT: track 53.4 -> 79.0 mm, vias 0 -> 2
- net /MCU/CELL_D_DISCHARGE: track 68.0 -> 92.6 mm, vias 2 -> 4
- net /MCU/CELL_D_DISCHARGE_CURRENT: track 45.9 -> 67.9 mm, vias 0 -> 2
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Other:
- net class Default: clearance 0.2 -> 0.15
- rule trace_clearance: 0.2 -> 0.15
- board text added: "Data"
- board text added: "Power"

Commit message: Soon...
Parts:
- added C615: 100n, Capacitor_SMD:C_0603_1608Metric, B.Cu at (189.0, 119.9)
- added C616: 100n, Capacitor_SMD:C_0603_1608Metric, B.Cu at (163.5, 103.3)
- added C717: 10u, Capacitor_SMD:C_0805_2012Metric, B.Cu at (113.0, 104.4)
- added C718: 10u, Capacitor_SMD:C_0805_2012Metric, B.Cu at (118.4, 113.2)
- added C719: 100n, Capacitor_SMD:C_0603_1608Metric, B.Cu at (126.1, 107.8)
- added C720: 100n, Capacitor_SMD:C_0603_1608Metric, B.Cu at (124.4, 108.2)
- added D606: D_Zener, Diode_SMD:D_SOD-123, B.Cu at (175.1, 96.7)
- added NT201: Net-Tie_2, NetTie:NetTie-2_SMD_Pad0.5mm, F.Cu at (102.2, 122.5)
- added NT301: Net-Tie_2, NetTie:NetTie-2_SMD_Pad0.5mm, F.Cu at (152.4, 122.5)
- added NT401: Net-Tie_2, NetTie:NetTie-2_SMD_Pad0.5mm, F.Cu at (167.8, 122.5)
- added NT501: Net-Tie_2, NetTie:NetTie-2_SMD_Pad0.5mm, F.Cu at (118.0, 122.7)
- added Q604: ZVN4206G, Package_TO_SOT_SMD:SOT-223-3_TabPin2, B.Cu at (168.7, 105.8)
- added Q605: ZVN4206G, Package_TO_SOT_SMD:SOT-223-3_TabPin2, B.Cu at (168.6, 95.2)
- added R627: 100k, Resistor_SMD:R_0603_1608Metric, B.Cu at (189.0, 118.4)
- added R628: 100k, Resistor_SMD:R_0603_1608Metric, B.Cu at (163.5, 106.4)
- added R629: 22k, Resistor_SMD:R_0603_1608Metric, B.Cu at (163.5, 107.9)
- added R630: 100, Resistor_SMD:R_0603_1608Metric, B.Cu at (163.5, 104.8)
- L201, L301, L401, L601: footprint Inductor_SMD:L_Wuerth_HCI-7050 -> Inductor_SMD:L_Wuerth_HCM-1052
- moved C409 18.8 mm to (184.1, 92.4), turned to 90 degrees
- moved C209 16.5 mm to (106.1, 96.3), turned to 0 degrees
- moved C309 16.4 mm to (156.7, 93.3), turned to 90 degrees
- moved C501 16.0 mm to (130.7, 96.5), turned to 0 degrees
- moved R418 15.1 mm to (179.7, 66.9), turned to 0 degrees
- moved R422 15.1 mm to (179.7, 65.4), turned to 180 degrees
- moved R408 15.1 mm to (164.7, 66.4)
- moved R308 15.0 mm to (140.4, 65.9)
- moved R208 14.8 mm to (90.5, 66.4)
- moved C404 14.7 mm to (165.8, 77.8), turned to 180 degrees
- moved R608 14.7 mm to (115.4, 66.5)
- moved C405 14.6 mm to (165.8, 75.8), turned to 180 degrees
- moved C604 14.5 mm to (115.3, 77.9), turned to 180 degrees
- moved C605 14.5 mm to (115.3, 76.0), turned to 180 degrees
- moved C304 14.4 mm to (140.7, 77.8), turned to 180 degrees
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Connections:
- J502 pad A1: GND -> GNDPWR
- J502 pad A12: GND -> GNDPWR
- J502 pad B1: GND -> GNDPWR
- J502 pad B12: GND -> GNDPWR
- J502 pad S1: GND -> /Power/SHIELD
- J601 pad 1: GND -> GNDPWR
- R222 pad 1: GNDPWR -> Net-(NT201-Pad2)
- R322 pad 1: GNDPWR -> Net-(NT301-Pad2)
- R422 pad 1: GNDPWR -> Net-(NT401-Pad2)
- R503 pad 1: GNDPWR -> Net-(NT501-Pad2)
- R626 pad 2: GND -> GNDPWR
- R701 pad 1: Net-(R701-Pad1) -> GND
- R701 pad 2: GND -> Net-(R701-Pad2)
- U202 pad 1: /MCU/CELL_A_VOLTAGE -> /MCU/CELL_A_CHARGE_CURRENT
- U202 pad 12: Net-(C206-Pad2) -> Net-(R214-Pad2)
- U202 pad 13: Net-(C206-Pad1) -> Net-(R218-Pad2)
- U202 pad 14: /MCU/CELL_A_CHARGE_CURRENT -> /MCU/CELL_A_VOLTAGE
- U202 pad 2: Net-(R218-Pad2) -> Net-(C206-Pad1)
- U202 pad 3: Net-(R214-Pad2) -> Net-(C206-Pad2)
- U302 pad 1: /MCU/CELL_C_VOLTAGE -> /MCU/CELL_C_CHARGE_CURRENT
- U302 pad 12: Net-(C306-Pad2) -> Net-(R314-Pad2)
- U302 pad 13: Net-(C306-Pad1) -> Net-(R318-Pad2)
- U302 pad 14: /MCU/CELL_C_CHARGE_CURRENT -> /MCU/CELL_C_VOLTAGE
- U302 pad 2: Net-(R318-Pad2) -> Net-(C306-Pad1)
- U302 pad 3: Net-(R314-Pad2) -> Net-(C306-Pad2)
- U402 pad 1: /MCU/CELL_D_VOLTAGE -> /MCU/CELL_D_DISCHARGE_CURRENT
- U402 pad 12: Net-(C406-Pad2) -> Net-(R414-Pad2)
- U402 pad 13: Net-(C406-Pad1) -> Net-(R418-Pad2)
- U402 pad 14: /MCU/CELL_D_DISCHARGE_CURRENT -> /MCU/CELL_D_VOLTAGE
- U402 pad 2: Net-(R418-Pad2) -> Net-(C406-Pad1)
- U402 pad 3: Net-(R414-Pad2) -> Net-(C406-Pad2)
- U502 pad 1: /MCU/CELL_B_VOLTAGE -> /MCU/CELL_B_CHARGE_CURRENT
- U502 pad 12: Net-(C606-Pad2) -> Net-(R502-Pad2)
- U502 pad 13: Net-(C606-Pad1) -> Net-(R503-Pad2)
- U502 pad 14: /MCU/CELL_B_CHARGE_CURRENT -> /MCU/CELL_B_VOLTAGE
- U502 pad 2: Net-(R503-Pad2) -> Net-(C606-Pad1)
- U502 pad 3: Net-(R502-Pad2) -> Net-(C606-Pad2)
- U701 pad 1: Net-(U701-Pad1) -> +3V3
- U701 pad 10: /MCU/CELL_A_DISCHARGE_CURRENT -> /MCU/CELL_A_VOLTAGE
- U701 pad 11: /MCU/CELL_A_TEMPERATURE -> /MCU/CELL_A_CHARGE_CURRENT
- U701 pad 14: /MCU/CELL_B_VOLTAGE -> /MCU/CELL_A_DISCHARGE_CURRENT
- U701 pad 21: /MCU/CELL_C_CHARGE_CURRENT -> /MCU/CELL_C_DISCHARGE_CURRENT
- U701 pad 22: /MCU/CELL_C_DISCHARGE_CURRENT -> /MCU/CELL_C_CHARGE_CURRENT
- U701 pad 27: /MCU/CELL_C_CHARGE -> Net-(U701-Pad27)
- U701 pad 38: /MCU/CELL_A_CHARGE -> /MCU/CELL_B_CHARGE
- U701 pad 39: /MCU/CELL_B_CHARGE -> /MCU/CELL_A_CHARGE
- U701 pad 58: /MCU/I2C_SCL -> Net-(U701-Pad58)
- U701 pad 59: /MCU/I2C_SDA -> /MCU/CELL_C_CHARGE
- U701 pad 60: Net-(R701-Pad1) -> Net-(R701-Pad2)
- U701 pad 61: Net-(U701-Pad61) -> /MCU/I2C_SCL
- U701 pad 62: Net-(U701-Pad62) -> /MCU/I2C_SDA
- U701 pad 8: /MCU/CELL_A_VOLTAGE -> /MCU/CELL_A_TEMPERATURE
- U701 pad 9: /MCU/CELL_A_CHARGE_CURRENT -> /MCU/CELL_B_TEMPERATURE
Routing:
- net GNDPWR: track 348.9 -> 140.9 mm, vias 93 -> 106
- net Net-(NT501-Pad2): track 0.00 -> 68.4 mm, vias 0 -> 1
- net Net-(NT401-Pad2): track 0.00 -> 66.7 mm, vias 0 -> 1
- net Net-(NT301-Pad2): track 0.00 -> 62.4 mm, vias 0 -> 1
- net Net-(NT201-Pad2): track 0.00 -> 61.2 mm, vias 0 -> 1
- net /CHARGE_POWER: track 86.2 -> 111.7 mm, vias 17 -> 20
- net /MCU/CELL_B_CHARGE_CURRENT: track 34.6 -> 59.4 mm
- net Net-(J601-Pad2): track 0.00 -> 23.3 mm, vias 0 -> 3
- net /MCU/CELL_A_VOLTAGE: track 88.2 -> 66.5 mm
- net /Power/SHIELD: track 0.00 -> 21.2 mm
- net /Power/USB_VBUS: track 50.7 -> 70.2 mm, vias 7 -> 9
- net /MCU/CELL_B_VOLTAGE: track 60.4 -> 42.6 mm, vias 2 -> 1
- net /MCU/CELL_C_VOLTAGE: track 47.1 -> 63.8 mm
- net /MCU/CELL_B_TEMPERATURE: track 5.16 -> 19.1 mm
- net /MCU/CELL_A_CHARGE: track 62.8 -> 49.0 mm
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Other:
- board text added: "GND TXD RXD"

Commit message: Soooooon...
Parts:
- removed C403, C615: 100n, Capacitor_SMD:C_0603_1608Metric
- removed the LOGO1 at (106.4, 111.3)
- removed R308: 22k 0.5%, Resistor_SMD:R_0603_1608Metric
- removed R627: 100k, Resistor_SMD:R_0603_1608Metric
- added C27: 100n, Capacitor_SMD:C_0603_1608Metric, B.Cu at (164.9, 60.8)
- added J3: Conn_01x02, Connector_JST:JST_EH_S2B-EH_1x02_P2.50mm_Horizontal, B.Cu at (161.1, 51.7)
- added JP1: SolderJumper_3_Open, Jumper:SolderJumper-3_P1.3mm_Open_Pad1.0x1.5mm_NumberLabels, B.Cu at (133.8, 133.3)
- added JP2: SolderJumper_3_Open, Jumper:SolderJumper-3_P1.3mm_Open_Pad1.0x1.5mm_NumberLabels, B.Cu at (136.2, 133.3)
- added LOGO1 (x2): Logo_Open_Hardware_Small, Symbol:OSHW-Logo_7.5x8mm_Copper, B.Cu at (106.4, 111.3)
- added Q15: Q_NMOS_GSD, Package_TO_SOT_SMD:SOT-23, B.Cu at (154.9, 71.8)
- added R108: 100, Resistor_SMD:R_0603_1608Metric, B.Cu at (154.8, 74.3)
- added R109: 100, Resistor_SMD:R_0603_1608Metric, B.Cu at (154.8, 75.9)
- added R19: 200m 1%, Resistor_SMD:R_1206_3216Metric, B.Cu at (98.7, 49.6)
- added R30: 200m 1%, Resistor_SMD:R_1206_3216Metric, B.Cu at (142.8, 73.8)
- added R39: 22k 0.5%, Resistor_SMD:R_0603_1608Metric, B.Cu at (141.9, 63.5)
- added R44: 200m 1%, Resistor_SMD:R_1206_3216Metric, B.Cu at (148.7, 49.6)
- added R5: 200m 1%, Resistor_SMD:R_1206_3216Metric, B.Cu at (92.8, 73.5)
- added R55: 200m 1%, Resistor_SMD:R_1206_3216Metric, B.Cu at (167.7, 73.7)
- added R69: 200m 1%, Resistor_SMD:R_1206_3216Metric, B.Cu at (173.7, 49.6)
- added R80: 200m 1%, Resistor_SMD:R_1206_3216Metric, B.Cu at (117.6, 73.7)
- added R94: 200m 1%, Resistor_SMD:R_1206_3216Metric, B.Cu at (123.7, 49.6)
- R20: renamed from R210; value 0R1 1% -> 200m 1%
- R31: renamed from R306; value 0R1 1% -> 200m 1%
- R45: renamed from R310; value 0R1 1% -> 200m 1%
- R56: renamed from R406; value 0R1 1% -> 200m 1%
- R6: renamed from R206; value 0R1 1% -> 200m 1%
- R70: renamed from R410; value 0R1 1% -> 200m 1%
- R81: renamed from R606; value 0R1 1% -> 200m 1%
- R95: renamed from R610; value 0R1 1% -> 200m 1%
- moved R54 3.75 mm to (176.3, 65.3)
- moved R53 3.74 mm to (176.3, 63.9)
- moved R89 3.44 mm to (116.7, 63.3), turned to 0 degrees
- moved R85 3.39 mm to (124.6, 56.5)
- moved R64 3.09 mm to (164.9, 63.3), turned to 0 degrees
- moved R60 3.00 mm to (173.3, 56.4), turned to 0 degrees
- moved C36 1.73 mm to (117.0, 60.8)
- moved R26 1.66 mm to (151.8, 67.3)
- moved R27 1.66 mm to (150.3, 67.3)
- moved R81 1.60 mm to (117.6, 71.4)
- moved R42 1.50 mm to (149.5, 58.0)
- moved R43 1.50 mm to (147.0, 57.2)
- moved R46 1.50 mm to (145.5, 57.2)
- moved R6 1.41 mm to (92.8, 71.2)
- moved R10 1.28 mm to (101.1, 56.5), turned to 0 degrees
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- renumbered BT201 to BT1, BT301 to BT2, BT401 to BT3, BT601 to BT4, C201 to C1, C301 to C10, C302 to C11, C304 to C12, C305 to C13, C306 to C14, C308 to C15, C309 to C16, C307 to C17, C303 to C18, C401 to C19, C202 to C2, C402 to C20, C404 to C21, C405 to C22, C406 to C23, C408 to C24, C409 to C25, C407 to C26, C601 to C28, C602 to C29, C204 to C3, C604 to C30, C605 to C31, C606 to C32, C608 to C33, C501 to C34, C607 to C35, C603 to C36, C609 to C37, C610 to C38, C616 to C39, C205 to C4, C612 to C40, C613 to C41, C611 to C42, C614 to C43, C713 to C44, C714 to C45, C708 to C46, C720 to C47, C715 to C48, C716 to C49, C206 to C5, C709 to C50, C711 to C51, C710 to C52, C717 to C53, C706 to C54, C718 to C55, C712 to C56, C701 to C57, C702 to C58, C703 to C59, C208 to C6, C704 to C60, C705 to C61, C707 to C62, C719 to C63, C209 to C7, C207 to C8, C203 to C9, D203 to D1, D603 to D10, D601 to D11, D602 to D12, D604 to D13, D605 to D14, D606 to D15, D608 to D16, D201 to D2, D202 to D3, D303 to D4, D301 to D5, D302 to D6, D403 to D7, D401 to D8, D402 to D9, J502 to J1, J601 to J2, J602 to J4, J701 to J5, J702 to J6, J703 to J7, L201 to L1, L301 to L2, L401 to L3, L601 to L4, NT201 to NT2, NT301 to NT3, NT401 to NT4, NT501 to NT5, Q201 to Q1, Q601 to Q10, Q603 to Q11, Q602 to Q12, Q604 to Q13, Q605 to Q14, Q203 to Q2, Q202 to Q3, Q301 to Q4, Q303 to Q5, Q302 to Q6, Q401 to Q7, Q403 to Q8, Q402 to Q9, R214 to R1, R213 to R10, R602 to R100, R620 to R101, R621 to R102, R622 to R103, R628 to R104, R630 to R105, R629 to R106, R626 to R107, R219 to R11, R625 to R110, R623 to R111, R624 to R112, R701 to R113, R702 to R114, R703 to R115, R220 to R12, R215 to R13, R208 to R14, R204 to R15, R203 to R16, R223 to R17, R211 to R18, R221 to R2, R212 to R21, R216 to R22, R209 to R23, R201 to R24, R202 to R25, R314 to R26, R321 to R27, R322 to R28, R318 to R29, R222 to R3, R305 to R32, R307 to R33, R317 to R34, R313 to R35, R319 to R36, R320 to R37, R315 to R38, R218 to R4, R304 to R40, R303 to R41, R323 to R42, R311 to R43, R312 to R46, R316 to R47, R309 to R48, R301 to R49, R302 to R50, R414 to R51, R421 to R52, R422 to R53, R418 to R54, R405 to R57, R407 to R58, R417 to R59, R413 to R60, R419 to R61, R420 to R62, R415 to R63, R408 to R64, R404 to R65, R403 to R66, R423 to R67, R411 to R68, R205 to R7, R412 to R71, R416 to R72, R409 to R73, R401 to R74, R402 to R75, R614 to R76, R502 to R77, R503 to R78, R618 to R79, R207 to R8, R605 to R82, R607 to R83, R617 to R84, R613 to R85, R619 to R86, R501 to R87, R615 to R88, R608 to R89, R217 to R9, R604 to R90, R603 to R91, R504 to R92, R611 to R93, R612 to R96, R616 to R97, R609 to R98, R601 to R99, TH201 to TH1, TH301 to TH2, TH401 to TH3, TH601 to TH4, TH701 to TH5, TH702 to TH6, TP601 to TP1, U202 to U1, U703 to U10, U704 to U11, U701 to U12, U702 to U13, U201 to U2, U302 to U3, U301 to U4, U402 to U5, U401 to U6, U502 to U7, U501 to U8, U602 to U9, Y701 to Y1
Connections:
- J4 pad 6: GND -> /Power/SHIELD2
- J6 pad 2: /MCU/RXD -> Net-(J6-Pad2)
- J6 pad 3: /MCU/TXD -> Net-(J6-Pad3)
- J7 pad 1: /MCU/TXD -> Net-(J6-Pad3)
- J7 pad 2: /MCU/RXD -> Net-(J6-Pad2)
Routing:
- net GND: track 323.2 -> 480.1 mm, vias 94 -> 135
- net Net-(J6-Pad3): track 0.00 -> 104.6 mm, vias 0 -> 1
- net Net-(J6-Pad2): track 0.00 -> 104.0 mm, vias 0 -> 1
- net /MCU/TXD: track 124.8 -> 29.1 mm, vias 1 -> 2
- net /MCU/RXD: track 124.7 -> 30.2 mm
- net /CHARGE_POWER: track 111.7 -> 152.2 mm, vias 20 -> 22
- net /MCU/CELL_C_CHARGE_CURRENT: track 70.3 -> 45.0 mm
- net Net-(J3-Pad2): track 0.00 -> 22.5 mm, vias 0 -> 2
- net /MCU/EN_FAN: track 0.00 -> 16.5 mm, vias 0 -> 1
- net /Power/SHIELD2: track 0.00 -> 11.9 mm, vias 0 -> 4
- net /MCU/CELL_D_VOLTAGE: track 72.6 -> 65.9 mm, vias 1 -> 2
- net /MCU/CELL_B_CHARGE_CURRENT: track 59.4 -> 65.7 mm
- net /MCU/CELL_D_DISCHARGE: track 89.7 -> 95.6 mm
- net Net-(R53-Pad2): track 9.79 -> 4.51 mm
- net /MCU/CELL_D_CHARGE_CURRENT: track 79.3 -> 75.1 mm, vias 2 -> 3
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- added copper zone on B.Cu, net GNDPWR
- added copper zone on B.Cu, net Net-(J2-Pad2)
Other:
- board text added: "Fan"
- board text added: "GND RXD TXD"
- board text added: "M"
- board text added: "S"
- board text removed: "GND TXD RXD"
