File: hw/v1/CellShaper.sch (KiCad schematic (older format))
At the start: 22 parts, among them J101 Conn_01x03, J102 Conn_01x03, J103 USB_B_Micro, J104 Screw_Terminal_01x02, J105 Conn_01x03, U101 TLV71333PDBV, U102 DAC084S085

Commit message: Progress with the schema and PCB....
Parts:
- removed C101, C102, C103, C104, C105, C106, C107, C108: 100n, Capacitor_SMD:C_0603_1608Metric, symbol Device:C
- removed J101, J102, J105: Conn_01x03, Connector_PinHeader_2.54mm:PinHeader_1x03_P2.54mm_Horizontal, symbol Connector_Generic:Conn_01x03
- removed J103: USB_B_Micro, Connector_USB:USB_Micro-B_Wuerth_629105150521, symbol Connector:USB_B_Micro
- removed J104: Screw_Terminal_01x02, TerminalBlock:TerminalBlock_bornier-2_P5.08mm, symbol Connector:Screw_Terminal_01x02
- removed R101, R102: R, symbol Device:R
- removed U101: TLV71333PDBV, Package_TO_SOT_SMD:SOT-23-5, symbol Regulator_Linear:TLV71333PDBV
- removed U102: DAC084S085, symbol Cell_Shaper:DAC084S085
- added H5, H6: M3 hole, MountingHole:MountingHole_3.2mm_M3_Pad, symbol Mechanical:MountingHole_Pad
- added LOGO1, LOGO2: Logo_Open_Hardware_Small, Symbol:OSHW-Logo_7.5x8mm_SilkScreen, symbol Graphic:Logo_Open_Hardware_Small
- added NT1: Net-Tie_2, NetTie:NetTie-2_SMD_Pad2.0mm, symbol Device:Net-Tie_2
- renumbered HS101 to HS1
Connections:
- net labels added: GNDA, GNDPWR
- net labels removed: +3V3, +5V, CELL_A_CHARGE, CELL_A_CHARGE_CURRENT, CELL_A_CHARGE_LED, CELL_A_DISCHARGE, CELL_A_DISCHARGE_CURRENT, CELL_A_DISCHARGE_LED, CELL_A_TEMPERATURE, CELL_A_VOLTAGE, CELL_B_CHARGE, CELL_B_CHARGE_CURRENT, CELL_B_CHARGE_LED, CELL_B_DISCHARGE, CELL_B_DISCHARGE_CURRENT, CELL_B_DISCHARGE_LED, CELL_B_TEMPERATURE, CELL_B_VOLTAGE, CELL_C_CHARGE, CELL_C_CHARGE_CURRENT, CELL_C_CHARGE_LED, CELL_C_DISCHARGE, CELL_C_DISCHARGE_LED, CELL_C_DISHARGE_CURRENT, CELL_C_TEMPERATURE, CELL_C_VOLTAGE, CELL_D_CHARGE, CELL_D_CHARGE_CURRENT, CELL_D_CHARGE_LED, CELL_D_DISCHARGE, CELL_D_DISCHARGE_CURRENT, CELL_D_DISCHARGE_LED, CELL_D_TEMPERATURE, CELL_D_VOLTAGE, DAC_DIN, DAC_SCLK, POWER_MEAS, RXD, SBWCLK, SBWDIO, TXD, USB_DN, USB_DP
- wire segments 107 -> 57
Other:
- note added: "Cell A"
- note added: "Cell B"
- note added: "Cell C"
- note added: "Cell D"
- note added: "MCU"
- note added: "Mounting holes"
- note added: "Power"
- note added: "STM32 here:\n- 19 ADC channels\n- 8 LEDs\n- 4 PWMs\n- USB-device\n- DAC SPI"
- note added: "TODO: Optional fan connector?"
- note removed: "STM32 here:\n- 17 ADC channels\n- 8 LEDs\n- 4 PWMs\n- USB-device\n- DAC SPI"
- moved on the sheet: H1, H2, H3, H4, HS1

Commit message: Progress...
Parts:
- LOGO1: footprint Symbol:OSHW-Logo_7.5x8mm_SilkScreen -> Symbol:OSHW-Logo_7.5x8mm_Copper
Connections:
- net GND: no longer HS1.1
- net GNDPWR: now also HS1.1
Changed lines of the file:
@@
-	1    0    0    -1
-$EndComp
-$Comp
-L power:GND #PWR0114
-U 1 1 5E9F736E
-P 1900 7100
-F 0 "#PWR0114" H 1900 6850 50  0001 C CNN
-F 1 "GND" H 1905 6927 50  0000 C CNN
-F 2 "" H 1900 7100 50  0001 C CNN
-F 3 "" H 1900 7100 50  0001 C CNN
-	1    1900 7100
 	1    0    0    -1
 $EndComp
@@
 F 0 "LOGO1" H 10300 7125 50  0001 C CNN
 F 1 "Logo_Open_Hardware_Small" H 10300 6625 50  0001 C CNN
-F 2 "Symbol:OSHW-Logo_7.5x8mm_SilkScreen" H 10300 6850 50  0001 C CNN
+F 2 "Symbol:OSHW-Logo_7.5x8mm_Copper" H 10300 6850 50  0001 C CNN
 F 3 "~" H 10300 6850 50  0001 C CNN
 	1    10300 6850
@@
 	1    0    0    -1
 $EndComp
+$Comp
+L power:GNDPWR #PWR0114
+U 1 1 5F3F0B4D
+P 1900 7100
+F 0 "#PWR0114" H 1900 6900 50  0001 C CNN
+F 1 "GNDPWR" H 1904 6946 50  0000 C CNN
+F 2 "" H 1900 7050 50  0001 C CNN
+F 3 "" H 1900 7050 50  0001 C CNN
+	1    1900 7100
+	1    0    0    -1
+$EndComp

Commit message: Soon...
Changed lines of the file:
@@
 F8 "~INT" B R 2600 2500 50
 F9 "CHARGE_VOLTAGE" O R 2600 1550 50
+F10 "EN_POWER" I R 2600 1650 50
 $EndSheet
 Wire Wire Line
@@
 F39 "I2C_~INT" I L 4150 2500 50
 F40 "CHARGE_VOLTAGE" I L 4150 1550 50
+F41 "EN_POWER" O L 4150 1650 50
 $EndSheet
 Text Notes 5300 3200 0    118  ~ 24
@@
 	1    0    0    -1
 $EndComp
+Wire Wire Line
+	4150 1650 2600 1650
 $EndSCHEMATC

Commit message: Soooooon...
Changed lines of the file:
@@
 $EndComp
 $Comp
-L power:GND #PWR0108
+L power:GND #PWR06
 U 1 1 5E926DBC
 P 5000 7250
-F 0 "#PWR0108" H 5000 7000 50  0001 C CNN
+F 0 "#PWR06" H 5000 7000 50  0001 C CNN
 F 1 "GND" H 5005 7077 50  0000 C CNN
 F 2 "" H 5000 7250 50  0001 C CNN
@@
 $EndComp
 $Comp
-L power:GND #PWR0109
+L power:GND #PWR07
 U 1 1 5E929CE7
 P 5200 7250
-F 0 "#PWR0109" H 5200 7000 50  0001 C CNN
+F 0 "#PWR07" H 5200 7000 50  0001 C CNN
 F 1 "GND" H 5205 7077 50  0000 C CNN
 F 2 "" H 5200 7250 50  0001 C CNN
@@
 $EndComp
 $Comp
-L power:GND #PWR0110
+L power:GND #PWR08
 U 1 1 5E929E85
 P 5400 7250
-F 0 "#PWR0110" H 5400 7000 50  0001 C CNN
+F 0 "#PWR08" H 5400 7000 50  0001 C CNN
 F 1 "GND" H 5405 7077 50  0000 C CNN
 F 2 "" H 5400 7250 50  0001 C CNN
@@
 $EndComp
 $Comp
-L power:GND #PWR0111
+L power:GND #PWR09
 U 1 1 5E92A041
 P 5600 7250
-F 0 "#PWR0111" H 5600 7000 50  0001 C CNN
+F 0 "#PWR09" H 5600 7000 50  0001 C CNN
 F 1 "GND" H 5605 7077 50  0000 C CNN
 F 2 "" H 5600 7250 50  0001 C CNN
@@
 $EndComp
 $Comp
-L power:GND #PWR0112
+L power:GND #PWR010
 U 1 1 5F00C100
 P 5800 7250
-F 0 "#PWR0112" H 5800 7000 50  0001 C CNN
+F 0 "#PWR010" H 5800 7000 50  0001 C CNN
 F 1 "GND" H 5805 7077 50  0000 C CNN
 F 2 "" H 5800 7250 50  0001 C CNN
@@
 $EndComp
 $Comp
-L power:GND #PWR0113
+L power:GND #PWR011
 U 1 1 5F00C2A7
 P 6000 7250
-F 0 "#PWR0113" H 6000 7000 50  0001 C CNN
+F 0 "#PWR011" H 6000 7000 50  0001 C CNN
 F 1 "GND" H 6005 7077 50  0000 C CNN
 F 2 "" H 6000 7250 50  0001 C CNN
@@
 CHARGE_POWER
 $Comp
-L power:GNDPWR #PWR0118
+L power:GNDPWR #PWR02
 U 1 1 5F391636
 P 1200 6700
-F 0 "#PWR0118" H 1200 6500 50  0001 C CNN
+F 0 "#PWR02" H 1200 6500 50  0001 C CNN
 F 1 "GNDPWR" H 1204 6546 50  0000 C CNN
 F 2 "" H 1200 6650 50  0001 C CNN
@@
 $EndComp
 $Comp
-L power:GND #PWR0119
+L power:GND #PWR01
 U 1 1 5F391EDC
 P 900 6700
-F 0 "#PWR0119" H 900 6450 50  0001 C CNN
+F 0 "#PWR01" H 900 6450 50  0001 C CNN
 F 1 "GND" H 905 6527 50  0000 C CNN
 F 2 "" H 900 6700 50  0001 C CNN
@@
 	900  6650 950  6650
 $Comp
-L power:GND #PWR0101
+L power:GND #PWR04
 U 1 1 5F53CCE5
 P 900 7250
-F 0 "#PWR0101" H 900 7000 50  0001 C CNN
+F 0 "#PWR04" H 900 7000 50  0001 C CNN
 F 1 "GND" H 905 7077 50  0000 C CNN
 F 2 "" H 900 7250 50  0001 C CNN
@@
 	900  7250 900  7200
 $Comp
-L power:GNDA #PWR0102
+L power:GNDA #PWR05
 U 1 1 5F54446F
 P 1200 7250
-F 0 "#PWR0102" H 1200 7000 50  0001 C CNN
+F 0 "#PWR05" H 1200 7000 50  0001 C CNN
 F 1 "GNDA" H 1205 7077 50  0000 C CNN
 F 2 "" H 1200 7250 50  0001 C CNN
@@
 F9 "CHARGE_VOLTAGE" O R 2600 1550 50
 F10 "EN_POWER" I R 2600 1650 50
+F11 "EN_FAN" I R 2600 1750 50
 $EndSheet
 Wire Wire Line
@@
 F40 "CHARGE_VOLTAGE" I L 4150 1550 50
 F41 "EN_POWER" O L 4150 1650 50
+F42 "EN_FAN" O L 4150 1750 50
 $EndSheet
 Text Notes 5300 3200 0    118  ~ 24
@@
 $EndComp
 $Comp
-L power:GNDPWR #PWR0114
+L power:GNDPWR #PWR03
 U 1 1 5F3F0B4D
 P 1900 7100
-F 0 "#PWR0114" H 1900 6900 50  0001 C CNN
+F 0 "#PWR03" H 1900 6900 50  0001 C CNN
 F 1 "GNDPWR" H 1904 6946 50  0000 C CNN
 F 2 "" H 1900 7050 50  0001 C CNN
@@
 Wire Wire Line
 	4150 1650 2600 1650
+Wire Wire Line
+	4150 1750 2600 1750
 $EndSCHEMATC
